File: radio.kicad_sch (KiCad schematic)
At the start: 21 parts, among them U2 4259-63

Commit message: add notes
Other:
- note added: "TOD: implement new chybechev filter"
Changed lines of the file:
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@@
+		)
+	)
+	(text "TOD: implement new chybechev filter"
+		(exclude_from_sim no)
+		(at 58.166 99.314 0)
+		(effects
+			(font
+				(size 1.27 1.27)
+			)
 		)
 	)
