File: RTLS_VIC.kicad_pcb (KiCad board)
At the start: 2 copper layers, 70 x 70 mm, 45 parts, among them J1 Conn_01x07_Socket, J3 Conn_01x03_Pin, J4 Conn_01x03_Pin, J5 Conn_01x03_Pin, J6 Conn_01x03_Pin, J7 Conn_01x04_Socket, J8 Conn_01x02_Pin, J9 Conn_01x07_Socket, SW1 TS-1187A-B-A-B, U1 AHT20-F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

Commit message: working on placements
Parts:
- added SW2: TS-1187A-B-A-B, lib:SW-SMD_4P-L5.1-W5.1-P3.70-LS6.5-TL_H1.5, F.Cu at (54.5, 48.0)
- moved C17 116.1 mm to (49.2, 99.1)
- moved C1 102.9 mm to (41.5, 110.0)
- moved C2 102.9 mm to (46.0, 110.0)
- moved C3 102.9 mm to (47.1, 110.0)
- moved U2 102.9 mm to (43.7, 110.5)
- moved L1 102.9 mm to (43.6, 107.1)
- moved R1 102.9 mm to (44.0, 114.7)
- moved R3 102.9 mm to (47.0, 113.2)
- moved C16 100.5 mm to (65.4, 96.3), turned to 90 degrees
- moved C15 100.5 mm to (69.8, 85.0)
- moved R11 100.4 mm to (90.2, 41.7)
- moved D1 98.7 mm to (86.9, 41.7)
- moved D2 98.7 mm to (86.9, 44.3)
- moved D3 98.7 mm to (86.9, 46.9)
- moved C12 94.5 mm to (68.4, 99.9), turned to -90 degrees
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Connections:
- U9 pad 39: unconnected-(U9-PC8-Pad39) -> DEBUG_BTN_1
Routing:
- added copper zone on B.Cu, net GND
- added copper zone on F.Cu, net GND

Commit message: nearly there
Parts:
- added C4: 4.7uF, Capacitor_SMD:C_0402_1005Metric, F.Cu at (144.3, 90.1)
- moved C1 107.5 mm to (143.1, 75.1), turned to 90 degrees
- moved L1 107.0 mm to (146.5, 77.6), turned to -90 degrees
- moved U2 104.7 mm to (143.1, 77.7), turned to 0 degrees
- moved C2 102.2 mm to (143.7, 79.9), turned to 180 degrees
- moved R1 101.7 mm to (138.9, 78.0), turned to 90 degrees
- moved C3 100.8 mm to (143.7, 81.0), turned to 180 degrees
- moved J2 99.1 mm to (155.9, 121.0), turned to -90 degrees
- moved R3 98.8 mm to (140.4, 81.0), turned to 90 degrees
- moved C17 94.9 mm to (143.0, 84.3), turned to 180 degrees
- moved SW2 80.1 mm to (127.7, 80.5), turned to -135 degrees
- moved D1 73.8 mm to (158.4, 59.8), turned to -90 degrees
- moved R11 71.6 mm to (158.5, 63.1), turned to -90 degrees
- moved D3 69.9 mm to (155.6, 59.9), turned to -90 degrees
- moved D2 67.6 mm to (152.7, 59.9), turned to -90 degrees
- moved R5 67.4 mm to (155.6, 63.0), turned to -90 degrees
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Connections:
- U6 pad 7: /Sensors/BMP581_INT -> BMP581_INT
- U8 pad 4: /Sensors/LSM6_INT1 -> LSM6_INT1
- U8 pad 9: /Sensors/LSM6_INT2 -> LSM6_INT2
- U9 pad 27: unconnected-(U9-PB1-Pad27) -> BMP581_INT
- U9 pad 28: unconnected-(U9-PB2-Pad28) -> LSM6_INT1
- U9 pad 29: unconnected-(U9-PB10-Pad29) -> LSM6_INT2
- U9 pad 30: unconnected-(U9-VCAP_1-Pad30) -> VCAP
Routing:
- net +3V3: track 0.00 -> 165.5 mm, vias 0 -> 5
- net +ESC_5V: track 0.00 -> 157.9 mm
- net SDA: track 0.00 -> 84.5 mm, vias 0 -> 4
- net SCL: track 0.00 -> 70.9 mm, vias 0 -> 2
- net PWM_4: track 0.00 -> 66.0 mm, vias 0 -> 1
- net PWM_2: track 0.00 -> 64.3 mm, vias 0 -> 1
- net SWCLK: track 0.00 -> 62.8 mm, vias 0 -> 4
- net DEBUG_TX: track 0.00 -> 54.9 mm, vias 0 -> 2
- net DEBUG_RX: track 0.00 -> 52.0 mm, vias 0 -> 2
- net SWDIO: track 0.00 -> 50.6 mm, vias 0 -> 2
- net BMP581_INT: track 0.00 -> 41.5 mm, vias 0 -> 2
- net RST: track 0.00 -> 34.5 mm
- net GND: track 0.00 -> 34.2 mm, vias 0 -> 52
- net LED_DEBUG_1: track 0.00 -> 31.4 mm, vias 0 -> 2
- net PWM_3: track 0.00 -> 30.7 mm, vias 0 -> 1
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- added copper zone on F.Cu, net +3V3
- added copper zone on F.Cu, net +ESC_5V
- added copper zone on F.Cu, net Net-(U2-LX1)
- added copper zone on F.Cu, net Net-(U2-LX2)
Other:
- board text added: "PWM_1"
- board text added: "PWM_2"
- board text added: "PWM_3"
- board text added: "PWM_4"
- board text added: "RESET"
- board text added: "SET POS"
- board text added: "VIC"

Commit message: preparing for prod
Parts:
- added G***: LOGO, LOGO, F.Cu at (180.1, 93.9)
- added J10: Conn_01x04_Socket, Connector_PinSocket_2.54mm:PinSocket_1x04_P2.54mm_Vertical, F.Cu at (164.7, 76.4)
- added J11: Conn_01x04_Socket, Connector_PinSocket_2.54mm:PinSocket_1x04_P2.54mm_Vertical, F.Cu at (166.2, 95.1)
- added J12: Conn_01x02_Pin, Connector_PinHeader_2.54mm:PinHeader_1x02_P2.54mm_Vertical, F.Cu at (143.2, 71.5)
- added J13: Conn_01x04_Socket, Connector_PinSocket_2.54mm:PinSocket_1x04_P2.54mm_Vertical, F.Cu at (127.0, 99.0)
- moved J9 3.65 mm to (154.6, 78.0)
- moved J1 3.54 mm to (157.1, 78.0)
- moved SW2 0.58 mm to (127.7, 80.0), turned to -90 degrees
Connections:
- U9 pad 24: unconnected-(U9-PC4-Pad24) -> DEBUG_NSS
- U9 pad 37: unconnected-(U9-PC6-Pad37) -> DEBUG_UART6_TX
- U9 pad 38: unconnected-(U9-PC7-Pad38) -> DEBUG_UART6_RX
Routing:
- net SPI_MOSI: track 0.00 -> 61.2 mm, vias 0 -> 2
- net SPI_MISO: track 0.00 -> 54.2 mm, vias 0 -> 2
- net SPI_SCK: track 0.00 -> 43.3 mm, vias 0 -> 2
- net DEBUG_NSS: track 0.00 -> 36.9 mm, vias 0 -> 1
- net +3V3: track 165.5 -> 201.1 mm
- net DEBUG_UART6_RX: track 0.00 -> 29.0 mm, vias 0 -> 1
- net DEBUG_UART6_TX: track 0.00 -> 26.2 mm, vias 0 -> 1
- net NSS: track 0.00 -> 21.7 mm, vias 0 -> 2
- net SCL: track 70.9 -> 85.9 mm
- net SDA: track 84.5 -> 96.3 mm, vias 4 -> 5
- net GND: track 34.2 -> 43.4 mm, vias 52 -> 69
Other:
- board text added: "Designed with love, Peter Cross | MAY 2025"
- board text added: "In Collab With: Jean-Raphael, Alanna, Jeanpierre, Julian"
- board text added: "RTLS BLACK"
- board text added: "jlcjlcjlcjlc"
