File: RTLS_VIC.kicad_pcb (KiCad board)
At the start: 2 copper layers, 70 x 70 mm, 52 parts, among them J1 Conn_01x07_Socket, J10 Conn_01x04_Socket, J11 Conn_01x04_Socket, J12 Conn_01x02_Pin, J13 Conn_01x04_Socket, J3 Conn_01x03_Pin, J4 Conn_01x03_Pin, J5 Conn_01x03_Pin, J6 Conn_01x03_Pin, J7 Conn_01x04_Socket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

Commit message: one more bom gen
Parts:
- moved G*** 0.62 mm to (180.1, 93.3)
Other:
- board text added: "VIC1"
- board text removed: "VIC"

Commit message: prod1
Parts:
- removed C27, C28: 100nF, Capacitor_SMD:C_0402_1005Metric
- removed U6: BMP581, lib:LGA-10_L2.0-W2.0-P0.50-TL_BMP581
- removed U8: LSM6DS3TR-C, lib:LGA-14_L3.0-W2.5-P0.50-TL
- added C5: 10nF, Capacitor_SMD:C_0402_1005Metric, F.Cu at (159.1, 98.8)
- added C6: 100nF, Capacitor_SMD:C_0402_1005Metric, F.Cu at (167.0, 80.7)
- added U3: ICM-42688-P, lib2:LGA-14_L3.0-W2.5-P0.50-TL, F.Cu at (156.2, 97.5)
- added U4: GZP6816D, lib2:SENSOR-SMD_XGZP6816D, F.Cu at (165.5, 82.5)
- J2: moved to B.Cu
- moved U1 1.51 mm to (168.5, 89.3)
Connections:
- U9 pad 27: BMP581_INT -> unconnected-(U9-PB1-Pad27)
Routing:
- net BMP581_INT: track 41.5 -> 0.00 mm, vias 2 -> 0
- net +3V3: track 201.1 -> 217.8 mm, vias 5 -> 8
- net SWCLK: track 62.8 -> 56.2 mm, vias 4 -> 3
- net LSM6_INT2: track 20.1 -> 24.7 mm
- net SWDIO: track 50.6 -> 54.7 mm, vias 2 -> 3
- net DEBUG_TX: track 54.9 -> 58.0 mm, vias 2 -> 3
- net RST: track 34.5 -> 37.4 mm, vias 0 -> 1
- net DEBUG_RX: track 52.0 -> 54.9 mm, vias 2 -> 3
- net GND: track 43.4 -> 40.7 mm, vias 69 -> 84
- net SDA: track 96.3 -> 95.0 mm
- net SCL: track 85.9 -> 87.1 mm
Other:
- board text added: "+"
- board text added: "3V3 GND"
- board text added: "3V3 SDA SCL GND"
- board text added: "3v3 TX RX GND"
- board text added: "GPS"
- board text added: "NSS SCK MISO MOSI"
- board text added: "UART6"

Commit message: sponsor and timing
Parts:
- added G***: LOGO, LOGO, B.Cu at (179.4, 92.2)
- added J14: Conn_01x03_Pin, Connector_PinHeader_2.54mm:PinHeader_1x03_P2.54mm_Vertical, F.Cu at (135.2, 67.3)
- added J15: Conn_01x03_Pin, Connector_PinHeader_2.54mm:PinHeader_1x03_P2.54mm_Vertical, F.Cu at (177.3, 67.9)
- added J16: Conn_01x03_Pin, Connector_PinHeader_2.54mm:PinHeader_1x03_P2.54mm_Vertical, F.Cu at (131.2, 114.0)
- added J17: Conn_01x03_Pin, Connector_PinHeader_2.54mm:PinHeader_1x03_P2.54mm_Vertical, F.Cu at (180.9, 114.0)
- moved J4 2.20 mm to (174.7, 70.5)
- moved J6 2.14 mm to (178.3, 111.4)
- moved J3 1.66 mm to (137.8, 69.9)
- moved J5 1.64 mm to (133.8, 111.4)
Connections:
- U9 pad 26: unconnected-(U9-PB0-Pad26) -> PWM_CH2_3
- U9 pad 27: unconnected-(U9-PB1-Pad27) -> PWM_CH2_4
- U9 pad 56: unconnected-(U9-PB4-Pad56) -> PWM_CH2_1
- U9 pad 57: unconnected-(U9-PB5-Pad57) -> PWM_CH2_2
Routing:
- net PWM_CH2_2: track 0.00 -> 72.5 mm, vias 0 -> 4
- net PWM_CH2_4: track 0.00 -> 54.2 mm, vias 0 -> 3
- net PWM_CH2_3: track 0.00 -> 40.1 mm, vias 0 -> 3
- net PWM_CH2_1: track 0.00 -> 26.9 mm
- net +ESC_5V: track 157.9 -> 164.9 mm
- net PWM_2: track 64.3 -> 61.0 mm
- net PWM_4: track 66.0 -> 63.1 mm
- net PWM_3: track 30.7 -> 29.6 mm
- net SPI_MISO: track 54.2 -> 55.2 mm
- net +3V3: track 217.8 -> 217.1 mm
- net LSM6_INT2: track 24.7 -> 24.0 mm
- net SWDIO: track 54.7 -> 55.3 mm
- net GND: track 40.7 -> 40.9 mm, vias 84 -> 79
Other:
- board text added: "Powered By:"
