File: RTLS_VIC.kicad_sch (KiCad schematic)
At the start: 41 parts, among them J10 Conn_01x04_Socket, J11 Conn_01x04_Socket, J12 Conn_01x02_Pin, J13 Conn_01x04_Socket, J14 Conn_01x03_Pin, J15 Conn_01x03_Pin, J16 Conn_01x03_Pin, J17 Conn_01x03_Pin, J8 Conn_01x02_Pin, SW1 TS-1187A-B-A-B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

Commit message: fix issues with power supply
Connections:
- net GND: now also U2.11 (EP), U2.4 (CFG2)
Changed lines of the file:
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@@
+	)
+	(junction
+		(at 257.81 83.82)
+		(diameter 0)
+		(color 0 0 0 0)
 	)
 	(junction
@@
 	)
 	(junction
+		(at 233.68 83.82)
+		(diameter 0)
+		(color 0 0 0 0)
+	)
+	(junction
 		(at 91.44 20.32)
 		(diameter 0)
@@
 	(wire
 		(pts
+			(xy 257.81 78.74) (xy 257.81 83.82)
+		)
+		(stroke
+			(width 0)
+			(type default)
+		)
+	)
+	(wire
+		(pts
 			(xy 20.32 177.8) (xy 22.86 177.8)
 		)
@@
 		)
 		(stroke
+			(width 0)
+			(type default)
+		)
+	)
+	(wire
+		(pts
+			(xy 233.68 81.28) (xy 233.68 83.82)
+		)
+		(stroke

Commit message: initial boom arm cad and sim
Other:
- note added: "in future revision, the PWM pins must go SIG POW GND"
Changed lines of the file:
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@@
+		)
+	)
+	(text "in future revision, the PWM pins must go SIG POW GND"
+		(exclude_from_sim no)
+		(at 170.18 124.206 0)
+		(effects
+			(font
+				(size 1.27 1.27)
+			)
 		)
 	)
